Commit message: open-loop effort gripper testing

File: gazebo_ros2_control_demos/urdf/gripper_effort_mimic_joint_sliding_base.xacro.urdf (robot description, URDF)
Before this commit: robot gripper, 4 links, 3 joints
Links:
- added link gripper_root_link, mass 1e3; collision box size=0.1 0.1 2.0; visual box size=0.1 0.1 2.0
- link base: geometry collision box size=1 1 0.5; visual box size=1 1 0.5
Joints:
- added joint base_prismatic: type prismatic, parent gripper_root_link, child base, origin xyz=0 0 0 rpy=0 0 0, axis 0 0 1, limit lower=0 upper=2 effort=1000.0 velocity=10
- joint world_fixed: child base -> gripper_root_link
